Commit message: 完成了物体的吸附以及容器尺寸的修改

File: cs612_moveit_config/config/cs612_suction_control.urdf.xacro (robot description, xacro)
@@ -111,5 +111,14 @@
     <child link="$(arg prefix)suction_cup_link" />
   </joint>
-  <link name="$(arg prefix)suction_tcp_link" />
+  <gazebo reference="$(arg prefix)wrist_3-suction_cup">
+    <preserveFixedJoint>true</preserveFixedJoint>
+  </gazebo>
+  <link name="$(arg prefix)suction_tcp_link">
+    <inertial>
+      <origin xyz="0 0 0" rpy="0 0 0" />
+      <mass value="0.001" />
+      <inertia ixx="1e-7" ixy="0" ixz="0" iyy="1e-7" iyz="0" izz="1e-7" />
+    </inertial>
+  </link>
   <joint name="$(arg prefix)suction_cup-tcp" type="fixed">
     <origin xyz="0 0 $(arg suction_tcp_offset_z)" rpy="0 0 0" />
@@ -117,8 +126,11 @@
     <child link="$(arg prefix)suction_tcp_link" />
   </joint>
+  <gazebo reference="$(arg prefix)suction_cup-tcp">
+    <preserveFixedJoint>false</preserveFixedJoint>
+  </gazebo>
   <gazebo>
     <plugin filename="ignition-gazebo-detachable-joint-system"
             name="ignition::gazebo::systems::DetachableJoint">
-      <parent_link>$(arg prefix)wrist_3_link</parent_link>
+      <parent_link>$(arg prefix)suction_cup_link</parent_link>
       <child_model>rect_pickup</child_model>
       <child_link>box_link</child_link>

Commit message: 基本完成了全流程

File: cs612_moveit_config/config/cs612_suction_control.urdf.xacro (robot description, xacro)
@@ -15,4 +15,9 @@
   <xacro:arg name="sim_ignition" default="true" />
   <xacro:arg name="simulation_controllers" default="" />
+  <xacro:arg name="controller_manager_name" default="controller_manager" />
+  <xacro:arg name="robot_param_node" default="robot_state_publisher" />
+  <xacro:arg name="suction_topic_ns" default="/cs612/suction" />
+  <xacro:arg name="base_origin_xyz" default="0 0 0" />
+  <xacro:arg name="base_origin_rpy" default="0 0 0" />
   <xacro:arg name="suction_tcp_offset_z" default="0.214" />
   <xacro:arg name="initial_positions_file" default="$(find eli_cs_robot_description)/config/initial_positions.yaml" />
@@ -41,5 +46,5 @@
     sim_ignition="$(arg sim_ignition)"
     initial_positions="${xacro.load_yaml(initial_positions_file)}">
-    <origin xyz="0 0 0" rpy="0 0 0" />
+    <origin xyz="$(arg base_origin_xyz)" rpy="$(arg base_origin_rpy)" />
   </xacro:cs_robot>
   <xacro:if value="$(arg sim_ignition)">
@@ -47,5 +52,7 @@
       <plugin filename="libign_ros2_control-system.so" name="ign_ros2_control::IgnitionROS2ControlPlugin">
         <parameters>$(arg simulation_controllers)</parameters>
-        <controller_manager_node_name>$(arg prefix)controller_manager</controller_manager_node_name>
+        <robot_param>robot_description</robot_param>
+        <robot_param_node>$(arg robot_param_node)</robot_param_node>
+        <controller_manager_name>$(arg controller_manager_name)</controller_manager_name>
       </plugin>
     </gazebo>
@@ -135,7 +142,7 @@
       <child_model>rect_pickup</child_model>
       <child_link>box_link</child_link>
-      <attach_topic>/cs612/suction/attach</attach_topic>
-      <detach_topic>/cs612/suction/detach</detach_topic>
-      <output_topic>/cs612/suction/state</output_topic>
+      <attach_topic>$(arg suction_topic_ns)/attach</attach_topic>
+      <detach_topic>$(arg suction_topic_ns)/detach</detach_topic>
+      <output_topic>$(arg suction_topic_ns)/state</output_topic>
     </plugin>
   </gazebo>
